File: hardware/EDA-Files/UP1-Progger/UP1-Progger.kicad_sch (KiCad schematic)
At the start: 11 parts, among them J1 UP1_Prog_Connector, J11 UP1_Prog_Connector, J2 USB_B_Micro, J4 SWD_Interface, J5 ST Link V2 Clone, SW1 Reset, SW2 Bootsel, U1 LDO_3V3_SOT23-3

Commit message: wip progger
Parts:
- added J3: Conn_01x03, Connector_PinHeader_2.54mm:PinHeader_1x03_P2.54mm_Vertical, symbol Connector_Generic:Conn_01x03
- U1: JLCPCB Rotation Offset 180 -> (none)
Connections:
- net +3.3V: now also J5.1 (Pin_1), J3.1 (Pin_1); no longer J5.7 (Pin_7), J5.8 (Pin_8)
- net +5V: now also J3.3 (Pin_3)
- net Bootsel: now also J5.8 (Pin_8)
- net D+: now also J5.3 (Pin_3)
- net D-: now also J5.4 (Pin_4)
- net GND: now also J5.10 (Pin_10); no longer J5.5 (Pin_5), J5.6 (Pin_6)
- net Reset: now also J5.7 (Pin_7); no longer J5.1 (Pin_1)
- net SWCLK: now also J5.5 (Pin_5); no longer J5.2 (Pin_2)
- net SWDIO: now also J5.6 (Pin_6); no longer J5.4 (Pin_4)
- new net: J3.2 (Pin_2), J5.2 (Pin_2)
